File: OxiKit-Brainboard_v1/OxiKit-Brainboard_v1.kicad_pcb (KiCad board)
At the start: 0 parts

Commit message: Component Placement - L1
Parts:
- added BZ1: Buzzer, Buzzer_Beeper:Buzzer_12x9.5RM7.6, F.Cu at (74.2, 90.0)
- added Brd1: SSD1306, SSD1306:128x64OLED, F.Cu at (117.0, 53.0)
- added C1: 220uF, Capacitor_THT:CP_Radial_D8.0mm_P3.50mm, F.Cu at (135.3, 70.0)
- added C2: 1uF, Capacitor_SMD:C_0805_2012Metric_Pad1.18x1.45mm_HandSolder, F.Cu at (147.0, 81.5)
- added C3: 1uF, Capacitor_SMD:C_0805_2012Metric_Pad1.18x1.45mm_HandSolder, F.Cu at (147.0, 77.8)
- added C4: 1uF, Capacitor_SMD:C_0805_2012Metric_Pad1.18x1.45mm_HandSolder, F.Cu at (147.0, 64.5)
- added C5: 1uF, Capacitor_SMD:C_0805_2012Metric_Pad1.18x1.45mm_HandSolder, F.Cu at (147.0, 94.8)
- added C6: 220uF, Capacitor_THT:CP_Radial_D8.0mm_P3.50mm, F.Cu at (135.3, 88.5)
- added C7: 100nF, Capacitor_SMD:C_0805_2012Metric_Pad1.18x1.45mm_HandSolder, F.Cu at (122.0, 73.2)
- added D1: LED, LED_SMD:LED_1206_3216Metric_Pad1.42x1.75mm_HandSolder, F.Cu at (138.8, 77.5)
- added D10: 1N4007, Diode_THT:D_DO-41_SOD81_P10.16mm_Horizontal, F.Cu at (119.9, 125.0)
- added D11: 1N4007, Diode_THT:D_DO-41_SOD81_P10.16mm_Horizontal, F.Cu at (130.1, 129.0)
- added D2: LED, LED_SMD:LED_1206_3216Metric_Pad1.42x1.75mm_HandSolder, F.Cu at (125.0, 99.8)
- added D3: 1N4007, Diode_THT:D_DO-41_SOD81_P10.16mm_Horizontal, F.Cu at (83.9, 125.0)
- added D4: 1N4007, Diode_THT:D_DO-41_SOD81_P10.16mm_Horizontal, F.Cu at (94.1, 129.0)
- added D5: LED, LED_SMD:LED_1206_3216Metric_Pad1.42x1.75mm_HandSolder, F.Cu at (107.0, 99.8)
- added D6: 1N4007, Diode_THT:D_DO-41_SOD81_P10.16mm_Horizontal, F.Cu at (101.9, 125.0)
- added D7: 1N4007, Diode_THT:D_DO-41_SOD81_P10.16mm_Horizontal, F.Cu at (112.1, 129.0)
- added D8: LED, LED_SMD:LED_1206_3216Metric_Pad1.42x1.75mm_HandSolder, F.Cu at (71.0, 99.2)
- added D9: LED, LED_SMD:LED_1206_3216Metric_Pad1.42x1.75mm_HandSolder, F.Cu at (89.0, 99.8)
- added H1: MountingHole, MountingHole:MountingHole_3.2mm_M3_Pad_Via, F.Cu at (55.0, 135.0)
- added H2: MountingHole, MountingHole:MountingHole_3.2mm_M3_Pad_Via, F.Cu at (55.0, 45.0)
- added H3: MountingHole, MountingHole:MountingHole_3.2mm_M3_Pad_Via, F.Cu at (145.0, 135.0)
- added H4: MountingHole, MountingHole:MountingHole_3.2mm_M3_Pad_Via, F.Cu at (145.0, 45.0)
- added J1: Jack-DC, Connector_BarrelJack:BarrelJack_Wuerth_6941xx301002, F.Cu at (135.7, 57.6)
- added J2: OXY-Sensor, Connector_JST:JST_XH_B2B-XH-A_1x02_P2.50mm_Vertical, F.Cu at (87.0, 45.0)
- added J3: Valve1, TerminalBlock:TerminalBlock_bornier-3_P5.08mm, F.Cu at (83.9, 136.0)
- added J4: Valve2, TerminalBlock:TerminalBlock_bornier-3_P5.08mm, F.Cu at (101.9, 136.0)
- added J5: UART, Connector_JST:JST_XH_B4B-XH-A_1x04_P2.50mm_Vertical, F.Cu at (72.8, 44.5)
- added J6: AC_IN, TerminalBlock:TerminalBlock_bornier-2_P5.08mm, F.Cu at (54.0, 116.5)
- added J7: I2C, Connector_JST:JST_XH_B4B-XH-A_1x04_P2.50mm_Vertical, F.Cu at (54.5, 81.2)
- added J8: Valve3, TerminalBlock:TerminalBlock_bornier-3_P5.08mm, F.Cu at (119.9, 136.0)
- added J9: Air Compresssor, TerminalBlock:TerminalBlock_bornier-2_P5.08mm, F.Cu at (69.5, 136.0)
- added K1: FINDER-36.11, Relay_THT:Relay_SPDT_Finder_36.11, F.Cu at (125.0, 104.0)
- added K2: FINDER-36.11, Relay_THT:Relay_SPDT_Finder_36.11, F.Cu at (107.0, 104.0)
- added K3: FINDER-36.11, Relay_THT:Relay_SPDT_Finder_36.11, F.Cu at (71.0, 104.0)
- added K4: FINDER-36.11, Relay_THT:Relay_SPDT_Finder_36.11, F.Cu at (89.0, 104.0)
- added R1: 1K, Resistor_SMD:R_0805_2012Metric_Pad1.20x1.40mm_HandSolder, F.Cu at (138.8, 80.0)
- added R2: 1K, Resistor_SMD:R_0805_2012Metric_Pad1.20x1.40mm_HandSolder, F.Cu at (112.0, 76.2)
- added R3: 10K, Resistor_SMD:R_0805_2012Metric_Pad1.20x1.40mm_HandSolder, F.Cu at (112.0, 72.0)
- added R4: 1K, Resistor_SMD:R_0805_2012Metric_Pad1.20x1.40mm_HandSolder, F.Cu at (119.5, 99.8)
- added R5: 1K, Resistor_SMD:R_0805_2012Metric_Pad1.20x1.40mm_HandSolder, F.Cu at (101.8, 99.8)
- added R6: 1K, Resistor_SMD:R_0805_2012Metric_Pad1.20x1.40mm_HandSolder, F.Cu at (65.8, 99.2)
- added R7: 1K, Resistor_SMD:R_0805_2012Metric_Pad1.20x1.40mm_HandSolder, F.Cu at (83.5, 99.8)
- added U1: Electron, particle:electron, F.Cu at (101.3, 63.0)
- added U2: LM7805_TO220, Package_TO_SOT_THT:TO-220-3_Vertical, F.Cu at (146.5, 68.5)
- added U3: LM7805_TO220, Package_TO_SOT_THT:TO-220-3_Vertical, F.Cu at (146.6, 85.5)
- added U4: LM358, Package_SO:SOIC-8_3.9x4.9mm_P1.27mm, F.Cu at (117.0, 74.0)
- added U5: ULN2003A, Package_DIP:DIP-16_W7.62mm_LongPads, F.Cu at (106.9, 86.2)
Other:
- board outline added: 100 x 100 mm
- copper layers 0 -> 2
