File: OxiKit-Brainboard_v1/OxiKit-Brainboard_v1.kicad_pcb (KiCad board)
At the start: 2 copper layers, 100 x 100 mm, 49 parts, among them J1 Jack-DC, J2 OXY-Sensor, J3 Valve1, J4 Valve2, J5 UART, J6 AC_IN, J7 I2C, J8 Valve3, J9 Air Compresssor, K1 FINDER-36.11, K2 FINDER-36.11, K3 FINDER-36.11, K4 FINDER-36.11, U1 Electron, U2 LM7805_TO220, U3 LM7805_TO220, U4 LM358, U5 ULN2003A

Commit message: Final routing
Parts:
- added D1: LED, LED_SMD:LED_1206_3216Metric_Pad1.42x1.75mm_HandSolder, F.Cu at (67.8, 84.8)
- added J4: Fan1, TerminalBlock:TerminalBlock_bornier-2_P5.08mm, F.Cu at (145.8, 58.5)
- added J5: Fan2, TerminalBlock:TerminalBlock_bornier-2_P5.08mm, F.Cu at (145.8, 71.0)
- added R10: 1K, Resistor_SMD:R_0805_2012Metric_Pad1.20x1.40mm_HandSolder, F.Cu at (82.2, 60.5)
- added R11: 1K, Resistor_SMD:R_0805_2012Metric_Pad1.20x1.40mm_HandSolder, F.Cu at (67.8, 90.0)
- added R3: 330R, Resistor_SMD:R_0805_2012Metric_Pad1.20x1.40mm_HandSolder, F.Cu at (67.8, 87.5)
- added R9: 1K, Resistor_SMD:R_0805_2012Metric_Pad1.20x1.40mm_HandSolder, F.Cu at (79.8, 60.5)
- added RN1: R_Network08, Resistor_THT:R_Array_SIP9, F.Cu at (109.7, 83.0)
- added SW1: Switch, Connector_JST:JST_XH_B2B-XH-A_1x02_P2.50mm_Vertical, F.Cu at (145.7, 81.8)
- added SW2: EmergencySW, Connector_JST:JST_XH_B2B-XH-A_1x02_P2.50mm_Vertical, F.Cu at (54.3, 86.5)
- added U5: TTGO-TCALL-SIM800, TTGO-TCALL-SIM800:TTGO-TCALL-SIM800, F.Cu at (103.0, 51.7)
- Brd1: moved to B.Cu
- moved J2 67.5 mm to (135.7, 125.1)
- moved C1 42.2 mm to (136.5, 112.2), turned to 90 degrees
- moved D12 38.0 mm to (92.1, 127.0)
- moved D11 38.0 mm to (82.0, 123.5)
- moved J10 38.0 mm to (82.0, 136.0)
- moved D5 34.1 mm to (128.1, 127.0)
- moved D4 34.0 mm to (117.9, 123.5)
- moved J7 34.0 mm to (117.9, 136.0)
- moved C4 23.5 mm to (145.1, 88.0)
- moved U3 23.5 mm to (144.6, 92.0)
- moved C3 23.3 mm to (145.1, 101.0)
- moved C2 22.6 mm to (145.0, 104.0)
- moved U4 22.6 mm to (144.6, 108.0)
- moved C6 22.3 mm to (145.0, 117.0)
- moved J6 15.8 mm to (54.3, 97.0)
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- renumbered C7 to C5, C5 to C6, C6 to C7, D9 to D10, D10 to D11, D11 to D12, D1 to D2, D2 to D3, D3 to D4, D4 to D5, D5 to D6, D6 to D7, D7 to D8, D8 to D9, J2 to J1, J8 to J10, J9 to J11, J1 to J2, J5 to J3, J7 to J6, J3 to J7, J4 to J8, J6 to J9, K4 to K3, K3 to K4, R2 to R1, R3 to R2, R1 to R4, R4 to R5, R5 to R6, R6 to R7, R7 to R8, U4 to U2, U2 to U3, U3 to U4, U5 to U6
Connections:
- C3 pad 1: +5V -> +5VP
- C6 pad 1: +5V -> +5VP
- C7 pad 1: +5V -> +5VP
- K1 pad 12: +V1/1 -> +V1/2
- K1 pad 14: +V1/2 -> +V1/1
- K2 pad 12: +V2/1 -> +V2/2
- K2 pad 14: +V2/2 -> +V2/1
- K3 pad 12: +V3/1 -> +V3/2
- K3 pad 14: +V3/2 -> +V3/1
- U1 pad 13: I6 -> I5
- U1 pad 14: I5 -> I4
- U1 pad 15: I4 -> I3
- U1 pad 16: I3 -> I2
- U1 pad 17: I2 -> I1
- U1 pad 18: I1 -> (no net)
- U1 pad 27: (no net) -> LED
- U1 pad 36: (no net) -> +3.3V
- U1 pad 6: (no net) -> EMR
- U3 pad 3: +5V -> +5VP
- U4 pad 3: +5V -> +5VP
- U6 pad 7: (no net) -> I7
Routing:
- net +5V: track 0.00 -> 307.0 mm, vias 0 -> 2
- net +3.3V: track 0.00 -> 225.9 mm, vias 0 -> 5
- net +12V: track 0.00 -> 172.9 mm
- net SCL: track 0.00 -> 125.1 mm, vias 0 -> 2
- net SDA: track 0.00 -> 120.4 mm
- net Oxy-out: track 0.00 -> 98.9 mm
- net LED: track 0.00 -> 89.4 mm, vias 0 -> 1
- net Net-(J1-Pad1): track 0.00 -> 86.9 mm
- net RX: track 0.00 -> 84.8 mm, vias 0 -> 2
- net TX: track 0.00 -> 77.3 mm, vias 0 -> 2
- net I5: track 0.00 -> 63.2 mm
- net +5VP: track 0.00 -> 54.7 mm
- net I4: track 0.00 -> 51.7 mm
- net I2: track 0.00 -> 37.2 mm
- net I3: track 0.00 -> 36.1 mm
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- added copper zone on B.Cu, net GND
- added copper zone on F.Cu, net GND
Other:
- outline, holes or cut-outs redrawn
- board text added: "2-Way Valve1"
- board text added: "2-Way Valve2"
- board text added: "2-Way Valve3"
- board text added: "AC IN"
- board text added: "Air Compressor"
- board text added: "FAN1"
- board text added: "FAN2"
- board text added: "GND"
- board text added: "I2C"
- board text added: "KE-25 OXY SENSOR"
- board text added: "L"
- board text added: "N"
- board text added: "SWITCH"
- board text added: "UART"
