File: OxiKit-Brainboard_v1/OxiKit-Brainboard_v1.kicad_sch (KiCad schematic)
At the start: 44 parts

Commit message: Component Placement - L1
Parts:
- added C7: 100nF, Capacitor_SMD:C_0805_2012Metric_Pad1.18x1.45mm_HandSolder, symbol Device:C_Small
- added H1, H2, H3, H4: MountingHole, MountingHole:MountingHole_3.2mm_M3_Pad_Via, symbol Mechanical:MountingHole
- added U1: Electron, particle:electron, symbol Particle-Devices:Electron
- BZ1: renamed from BZ?; footprint (none) -> Buzzer_Beeper:Buzzer_12x9.5RM7.6
- Brd1: renamed from Brd?; footprint (none) -> SSD1306:128x64OLED
- C1, C6: renamed from C?; footprint (none) -> Capacitor_THT:CP_Radial_D8.0mm_P3.50mm
- C2, C3, C4, C5: renamed from C?; footprint (none) -> Capacitor_SMD:C_0805_2012Metric_Pad1.18x1.45mm_HandSolder
- D1, D2, D5, D8, D9: renamed from D?; footprint (none) -> LED_SMD:LED_1206_3216Metric_Pad1.42x1.75mm_HandSolder
- J1: renamed from J?; footprint (none) -> Connector_BarrelJack:BarrelJack_Wuerth_6941xx301002
- J2: renamed from J?; footprint (none) -> Connector_JST:JST_XH_B2B-XH-A_1x02_P2.50mm_Vertical
- J3, J4, J8: renamed from J?; footprint (none) -> TerminalBlock:TerminalBlock_bornier-3_P5.08mm
- J5, J7: renamed from J?; footprint (none) -> Connector_JST:JST_XH_B4B-XH-A_1x04_P2.50mm_Vertical
- J6, J9: renamed from J?; footprint (none) -> TerminalBlock:TerminalBlock_bornier-2_P5.08mm
- R1, R2, R3, R4, R5, R6, R7: renamed from R?; footprint (none) -> Resistor_SMD:R_0805_2012Metric_Pad1.20x1.40mm_HandSolder
- U5: renamed from U?; footprint (none) -> Package_DIP:DIP-16_W7.62mm_LongPads
- gave numbers to parts that had none: 13
Connections:
- net 3.3V is gone; now on net +3.3V: Brd1.2 (VCC)
- net +5V: now also J7.1 (Pin_1), C7.1, U1.1 (VIN)
- net +V1/1: now also D3.1 (K), J3.1 (Pin_1)
- net +V1/2: now also D4.1 (K), J3.3 (Pin_3)
- net +V2/1: now also D6.1 (K)
- net +V2/2: now also D7.1 (K)
- net +V3/2: now also D11.1 (K); no longer J8.1 (Pin_1), K4.12
- net GND: now also J5.4 (Pin_4), J7.4 (Pin_4), C7.2, U1.2 (GND), U1.33 (GND)
- net I1: now also U1.18 (B0)
- net I2: now also U1.17 (B1)
- net I3: now also U1.16 (B2)
- net I4: now also U1.15 (B3)
- net I5: now also U1.14 (B4)
- net I6: now also U1.13 (B5)
- net O1: no longer D5.2 (A), D8.2 (A), D9.2 (A), K2.A2, K3.A2, K4.A2
- net O2: now also D5.2 (A), K2.A2
- net O3: now also D9.2 (A), K4.A2
- net O4: now also D8.2 (A), K3.A2
- net Oxy-out: now also U1.12 (A0)
- net SCL: now also J5.3 (Pin_3), U1.26 (D1)
- net SDA: now also J5.2 (Pin_2), U1.25 (D0)
- net TX: now reaches J7.2 (Pin_2)
- net TX: now also U1.3 (TX)
- net RX: now reaches J7.3 (Pin_3)
- net RX: now also U1.4 (RX)
- net +3.3V: now reaches J5.1 (Pin_1)
- removed net +V1-1: D10.1 (K), D3.1 (K), D6.1 (K), J3.1 (Pin_1)
- removed net +V1-2: D11.1 (K), D4.1 (K), D7.1 (K), J3.3 (Pin_3)
- new net +3V3: U1.36 (3V3)
- new net +V3/1: D10.1 (K), J8.1 (Pin_1), K4.12
Other:
- note added: "Particle Electron"
- moved on the sheet: J2, J5, R2, R3, U4A, U4C

Commit message: Final routing
Parts:
- added D1: LED, LED_SMD:LED_1206_3216Metric_Pad1.42x1.75mm_HandSolder, symbol Device:LED
- added J4: Fan1, TerminalBlock:TerminalBlock_bornier-2_P5.08mm, symbol Connector_Generic:Conn_01x02
- added J5: Fan2, TerminalBlock:TerminalBlock_bornier-2_P5.08mm, symbol Connector_Generic:Conn_01x02
- added R10, R11, R9: 1K, Resistor_SMD:R_0805_2012Metric_Pad1.20x1.40mm_HandSolder, symbol Device:R_Small
- added R3: 330R, Resistor_SMD:R_0805_2012Metric_Pad1.20x1.40mm_HandSolder, symbol Device:R_Small
- added RN1: R_Network08, Resistor_THT:R_Array_SIP9, symbol Device:R_Network08
- added SW1: Switch, Connector_JST:JST_XH_B2B-XH-A_1x02_P2.50mm_Vertical, symbol Switch:SW_DIP_x01
- added SW2: EmergencySW, Connector_JST:JST_XH_B2B-XH-A_1x02_P2.50mm_Vertical, symbol Switch:SW_DIP_x01
- added U5: TTGO-TCALL-SIM800, TTGO-TCALL-SIM800:TTGO-TCALL-SIM800, symbol electroShri:TTGO-TCALL-SIM800
- renumbered C7 to C5, C5 to C6, C6 to C7, D9 to D10, D10 to D11, D11 to D12, D1 to D2, D2 to D3, D3 to D4, D4 to D5, D5 to D6, D6 to D7, D7 to D8, D8 to D9, J2 to J1, J8 to J10, J9 to J11, J1 to J2, J5 to J3, J7 to J6, J3 to J7, J4 to J8, J6 to J9, K4 to K3, K3 to K4, R2 to R1, R3 to R2, R1 to R4, R4 to R5, R5 to R6, R6 to R7, R7 to R8, U4 to U2, U2 to U3, U3 to U4, U5 to U6
Connections:
- net +3V3 is gone; now on net +3.3V: U1.36 (3V3)
- net +12V: now also J4.1 (Pin_1), J5.1 (Pin_1)
- net +3.3V: now also R10.1, R11.2, R9.1, U5.1 (3V3)
- net +5V: now also SW1.2, U5.19 (5V); no longer C3.1, C6.1, C7.1, U3.3 (VO), U4.3 (VO)
- net +V1/1: now also K1.14; no longer K1.12
- net +V1/2: now also K1.12; no longer K1.14
- net +V2/1: now also K2.14; no longer K2.12
- net +V2/2: now also K2.12; no longer K2.14
- net +V3/1: now also K3.14; no longer K3.12
- net +V3/2: now also K3.12; no longer K3.14
- net GND: now also J4.2 (Pin_2), J5.2 (Pin_2), R3.2, RN1.1 (common), SW2.1, U5.14 (GND), U5.22 (GND), U5.28 (GND)
- net I1: now also U1.17 (B1), RN1.2 (R1), U5.23 (GPIO23); no longer U1.18 (B0)
- net I2: now also U1.16 (B2), RN1.3 (R2), U5.29 (GPIO19); no longer U1.17 (B1)
- net I3: now also U1.15 (B3), RN1.4 (R3), U5.30 (GPIO18); no longer U1.16 (B2)
- net I4: now also U1.14 (B4), RN1.5 (R4), U5.34 (GPIO4); no longer U1.15 (B3)
- net I5: now also U1.13 (B5), RN1.6 (R5), U5.36 (GPIO2); no longer U1.14 (B4)
- net I6: now also RN1.7 (R6); no longer U1.13 (B5)
- net I7: now also RN1.8 (R7)
- net Oxy-out: now also U5.5 (GPIO34)
- net RX: now also U5.12 (GPIO14)
- net SCL: now also R9.2, U5.24 (GPIO22)
- net SDA: now also R10.2, U5.27 (GPIO21)
- net TX: now also U5.13 (GPIO12)
- net LED: now reaches U1.27 (D2)
- net LED: now also D1.2 (A), U5.31 (GPIO5)
- net EMR: now reaches U1.6 (A6)
- net EMR: now also R11.1, SW2.2, U5.37 (GPIO15)
- new net: D1.1 (K), R3.1
- new net +5VP: C3.1, C6.1, C7.1, SW1.1, U3.3 (VO), U4.3 (VO)
- no-connect marks 0 -> 6
Other:
- note added: "ESP32 + SIM800"
- note added: "Fan"
- note added: "I2C Pullups"
- note added: "Indication LED"
- moved on the sheet: BZ1, Brd1, C1, C2, C3, C4, C5, C6, C7, D10, D11, D12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
